File: Lab3_project.kicad_sch (KiCad schematic)
At the start: 39 parts, among them J1 POWER IN, J2 PROG, J3 Conn_Coaxial, SW2 RESET, SW3 BOOT, U1 STM32F407IGTx, U2 AMS1117-3.3, U3 CAT24C256, U4 MPU-6000, U5 NEO-M8N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

Commit message: Trace route
Parts:
- U3: footprint Package_DIP:DIP-8_W7.62mm_Socket -> Package_SO:SOIC-8_3.9x4.9mm_P1.27mm
Other:
- moved on the sheet: C11
Changed lines of the file:
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@@
 	(wire
 		(pts
-			(xy 355.6 198.12) (xy 360.68 198.12)
+			(xy 355.6 198.12) (xy 359.41 198.12)
 		)
 		(stroke
@@
 	(wire
 		(pts
-			(xy 368.3 198.12) (xy 370.84 198.12)
+			(xy 367.03 198.12) (xy 370.84 198.12)
 		)
 		(stroke
@@
 			)
 		)
-		(property "Footprint" "Package_DIP:DIP-8_W7.62mm_Socket"
+		(property "Footprint" "Package_SO:SOIC-8_3.9x4.9mm_P1.27mm"
 			(at 358.14 114.3 0)
 			(effects
@@
 	(symbol
 		(lib_id "Device:C")
-		(at 364.49 198.12 90)
+		(at 363.22 198.12 90)
 		(unit 1)
 		(exclude_from_sim no)
@@
 		(dnp no)
 		(property "Reference" "C11"
-			(at 364.49 203.2 90)
+			(at 363.22 203.2 90)
 			(effects
 				(font
@@
 		)
 		(property "Value" "22 pF"
-			(at 364.49 205.74 90)
+			(at 363.22 205.74 90)
 			(effects
 				(font
@@
 		)
 		(property "Footprint" "Capacitor_SMD:C_0805_2012Metric_Pad1.18x1.45mm_HandSolder"
-			(at 368.3 197.1548 0)
+			(at 367.03 197.1548 0)
 			(effects
 				(font
@@
 		)
 		(property "Datasheet" "~"
-			(at 364.49 198.12 0)
+			(at 363.22 198.12 0)
 			(effects
 				(font
@@
 		)
 		(property "Description" "Unpolarized capacitor"
-			(at 364.49 198.12 0)
-			(effects
-				(font
+			(at 363.22 198.12 0)
+			(effects
+				(font
