File: Lab3_project.kicad_pcb (KiCad board)
At the start: 2 copper layers, 33 parts, among them J1 POWER IN, J2 PROG, J3 Conn_Coaxial, SW2 RESET, SW3 BOOT, U1 STM32F407IGTx, U2 AMS1117-3.3, U3 CAT24C256, U4 MPU-6000, U5 NEO-M8N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

Commit message: Trace route
Parts:
- added C11: 22 pF, Capacitor_SMD:C_0805_2012Metric_Pad1.18x1.45mm_HandSolder, F.Cu at (74.9, 120.4)
- added C19: 0.1 uF, Capacitor_SMD:C_0805_2012Metric_Pad1.18x1.45mm_HandSolder, F.Cu at (96.3, 106.7)
- added C20: 0.1 uF, Capacitor_SMD:C_0805_2012Metric_Pad1.18x1.45mm_HandSolder, F.Cu at (68.3, 91.3)
- added C21: 2.2 nF, Capacitor_SMD:C_0805_2012Metric_Pad1.18x1.45mm_HandSolder, F.Cu at (69.8, 79.2)
- added C22: 0.1 uF, Capacitor_SMD:C_0805_2012Metric_Pad1.18x1.45mm_HandSolder, F.Cu at (73.5, 80.1)
- added C23: 0.1 uF, Capacitor_SMD:C_0805_2012Metric_Pad1.18x1.45mm_HandSolder, F.Cu at (118.6, 85.7)
- L1: value 28 uH -> 33 nH
- U3: footprint Package_DIP:DIP-8_W7.62mm_Socket -> Package_SO:SOIC-8_3.9x4.9mm_P1.27mm
- moved C17 94.2 mm to (75.5, 91.9), turned to 180 degrees
- moved C18 92.0 mm to (77.6, 96.1), turned to -90 degrees
- moved C4 83.2 mm to (82.7, 101.8), turned to 180 degrees
- moved C15 79.9 mm to (93.9, 68.3), turned to 180 degrees
- moved J3 75.6 mm to (66.6, 109.0)
- moved C6 74.7 mm to (90.8, 101.8)
- moved J2 74.0 mm to (69.0, 68.6), turned to 90 degrees
- moved Y1 72.3 mm to (92.8, 63.0), turned to 180 degrees
- moved C14 72.2 mm to (101.1, 68.3)
- moved L1 69.8 mm to (74.9, 117.2), turned to 180 degrees
- moved C7 68.9 mm to (96.3, 101.8)
- moved C2 66.8 mm to (86.4, 57.2), turned to 180 degrees
- moved C3 66.3 mm to (97.1, 131.6), turned to 90 degrees
- moved C8 62.1 mm to (102.8, 101.8)
- moved R9 59.6 mm to (109.5, 55.6), turned to 90 degrees
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Connections:
- J3 pad 1: unconnected-(J3-In-Pad1) -> Net-(J3-In)
- J3 pad 2: unconnected-(J3-Ext-Pad2) -> GND
- L1 pad 1: unconnected-(L1-Pad1) -> Net-(U5-VCC_RF)
- L1 pad 2: unconnected-(L1-Pad2) -> Net-(J3-In)
- R1 pad 2: unconnected-(R1-Pad2) -> I2C_SCL
- R2 pad 2: unconnected-(R2-Pad2) -> I2C_SDA
- U3 pad 1: unconnected-(U3-A0-Pad1) -> GND
- U3 pad 2: unconnected-(U3-A1-Pad2) -> GND
- U3 pad 3: unconnected-(U3-A2-Pad3) -> GND
- U3 pad 4: unconnected-(U3-GND-Pad4) -> GND
- U3 pad 5: unconnected-(U3-SDA-Pad5) -> I2C_SDA
- U3 pad 6: unconnected-(U3-SCL-Pad6) -> I2C_SCL
- U3 pad 7: unconnected-(U3-WP-Pad7) -> MEM_WP
- U3 pad 8: unconnected-(U3-VCC-Pad8) -> +3.3V
- U4 pad 1: unconnected-(U4-CLKIN-Pad1) -> GND
- U4 pad 10: unconnected-(U4-REGOUT-Pad10) -> Net-(U4-REGOUT)
- U4 pad 11: unconnected-(U4-FSYNC-Pad11) -> GND
- U4 pad 13: unconnected-(U4-VDD-Pad13) -> +3.3V
- U4 pad 18: unconnected-(U4-GND-Pad18) -> GND
- U4 pad 20: unconnected-(U4-CPOUT-Pad20) -> Net-(U4-CPOUT)
- U4 pad 23: unconnected-(U4-SCL/SCLK-Pad23) -> SPI_SCK
- U4 pad 24: unconnected-(U4-SDA/MOSI-Pad24) -> SPI_MOSI
- U4 pad 8: unconnected-(U4-~{CS}-Pad8) -> SPI_CS
- U4 pad 9: unconnected-(U4-AD0/MISO-Pad9) -> SPI_MISO
- U5 pad 11: unconnected-(U5-RF_IN-Pad11) -> Net-(U5-RF_IN)
- U5 pad 9: unconnected-(U5-VCC_RF-Pad9) -> Net-(U5-VCC_RF)
Routing:
- net +3.3V: track 0.00 -> 485.6 mm, vias 0 -> 3
- net NRST: track 0.00 -> 88.2 mm
- net SWDIO: track 0.00 -> 46.0 mm, vias 0 -> 1
- net SWCLK: track 0.00 -> 42.7 mm
- net SWO: track 0.00 -> 42.3 mm, vias 0 -> 2
- net BOOT: track 0.00 -> 36.2 mm
- net +5V: track 0.00 -> 33.0 mm
- net SPI_CS: track 0.00 -> 31.9 mm, vias 0 -> 2
- net SPI_MISO: track 0.00 -> 25.7 mm
- net SPI_SCK: track 0.00 -> 25.6 mm
- net SPI_MOSI: track 0.00 -> 25.6 mm
- net Net-(J3-In): track 0.00 -> 22.5 mm
- net I2C_SCL: track 0.00 -> 21.9 mm
- net UART_RX: track 0.00 -> 21.2 mm
- net UART_TX: track 0.00 -> 19.9 mm
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- added copper zone on B.Cu, net GND
- added copper zone on F.Cu, net GND
Other:
- board outline added: 67 x 87 mm
- board text added: "Created by Мегатіма #3"

Commit message: fix gnd zone
Parts:
- moved C1 53.2 mm to (147.3, 62.7)
- moved C11 53.2 mm to (127.8, 125.9)
- moved C13 53.2 mm to (168.5, 119.5)
- moved C14 53.2 mm to (154.0, 73.7)
- moved C16 53.2 mm to (164.1, 111.5)
- moved C19 53.2 mm to (149.3, 112.2)
- moved C2 53.2 mm to (139.3, 62.7)
- moved C21 53.2 mm to (122.7, 84.7)
- moved C22 53.2 mm to (126.5, 85.6)
- moved C23 53.2 mm to (171.6, 91.2)
- moved C4 53.2 mm to (135.6, 107.3)
- moved J1 53.2 mm to (138.5, 134.5)
- moved J3 53.2 mm to (119.6, 114.5)
- moved L1 53.2 mm to (127.8, 122.7)
- moved R1 53.2 mm to (169.8, 96.7)
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